Commit message: reorder STLs

File: glove/model/glove_non_diametric.urdf (robot description, URDF)
Before this commit: robot glove_non_diametric, 129 links, 128 joints
Links:
- link _dip_2: geometry visual mesh filename=package://glove_non_diametric/meshes/printed/DIP/_dip_2.stl scale=1 1 1
- link _dip_2_1: geometry visual mesh filename=package://glove_non_diametric/meshes/printed/DIP/_dip_2.stl scale=1 1 1
- link bottom_base: geometry visual mesh filename=package://glove_non_diametric/meshes/printed/palm/bottom_ba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 scale=1 1 1
- link broached_hexagon_socket_head_cap_screw_asme_b18_3_1m___m2x0_4_x_6_steel_grade_2_plain: geometry visual mesh filename=package://glove_non_diametric/meshes/hardware/Broached_Hexa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 scale=1 1 1
- link broached_hexagon_socket_head_cap_screw_asme_b18_3_1m___m2x0_4_x_6_steel_grade_2_plain__1_: geometry visual mesh filename=package://glove_non_diametric/meshes/hardware/Broached_Hexa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 scale=1 1 1
- link broached_hexagon_socket_head_cap_screw_asme_b18_3_1m___m2x0_4_x_6_steel_grade_2_plain__2_: geometry visual mesh filename=package://glove_non_diametric/meshes/hardware/Broached_Hexa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 scale=1 1 1
- link broached_hexagon_socket_head_cap_screw_asme_b18_3_1m___m2x0_4_x_6_steel_grade_2_plain__3_: geometry visual mesh filename=package://glove_non_diametric/meshes/hardware/Broached_Hexa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 scale=1 1 1
- link broached_hexagon_socket_head_cap_screw_asme_b18_3_1m___m2x0_4_x_6_steel_grade_2_plain__4_: geometry visual mesh filename=package://glove_non_diametric/meshes/hardware/Broached_Hexa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 scale=1 1 1
- link broached_hexagon_socket_head_cap_screw_asme_b18_3_1m___m2x0_4_x_6_steel_grade_2_plain__5_: geometry visual mesh filename=package://glove_non_diametric/meshes/hardware/Broached_Hexa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 scale=1 1 1
- link broached_hexagon_socket_head_cap_screw_asme_b18_3_1m___m2x0_4_x_6_steel_grade_2_plain__6_: geometry visual mesh filename=package://glove_non_diametric/meshes/hardware/Broached_Hexa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 scale=1 1 1
- link broached_hexagon_socket_head_cap_screw_asme_b18_3_1m___m2x0_4_x_6_steel_grade_2_plain__7_: geometry visual mesh filename=package://glove_non_diametric/meshes/hardware/Broached_Hexa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 scale=1 1 1
- link broached_hexagon_socket_head_cap_screw_asme_b18_3_1m___m2x0_4_x_6_steel_grade_2_plain__8_: geometry visual mesh filename=package://glove_non_diametric/meshes/hardware/Broached_Hexa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 scale=1 1 1
- link broached_hexagon_socket_head_cap_screw_asme_b18_3_1m___m2x0_4_x_6_steel_grade_2_plain__9_: geometry visual mesh filename=package://glove_non_diametric/meshes/hardware/Broached_Hexa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 scale=1 1 1
- link desk_display_pcb__1_: geometry visual mesh filename=package://glove_non_diametric/meshes/electronics/desk_displ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 scale=1 1 1
- link dip_1: geometry visual mesh filename=package://glove_non_diametric/meshes/printed/DIP/dip_1.stl scale=1 1 1
- link dip_1_1: geometry visual mesh filename=package://glove_non_diametric/meshes/printed/DIP/dip_1.stl scale=1 1 1
- link dip_1_2: geometry visual mesh filename=package://glove_non_diametric/meshes/printed/DIP/dip_1.stl scale=1 1 1
- link dip_1_3: geometry visual mesh filename=package://glove_non_diametric/meshes/printed/DIP/dip_1.stl scale=1 1 1
- link dip_1_4: geometry visual mesh filename=package://glove_non_diametric/meshes/printed/DIP/dip_1.stl scale=1 1 1
- link dip_1_5: geometry visual mesh filename=package://glove_non_diametric/meshes/printed/DIP/dip_1.stl scale=1 1 1
- link hexagon_socket_head_cap_screw_iso_4762___m2_x_10_steel_4_6_plain: geometry visual mesh filename=package://glove_non_diametric/meshes/hardware/Hexagon_Socke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 scale=1 1 1
- link hexagon_socket_head_cap_screw_iso_4762___m2_x_10_steel_4_6_plain__10_: geometry visual mesh filename=package://glove_non_diametric/meshes/hardware/Hexagon_Socke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 scale=1 1 1
- link hexagon_socket_head_cap_screw_iso_4762___m2_x_10_steel_4_6_plain__11_: geometry visual mesh filename=package://glove_non_diametric/meshes/hardware/Hexagon_Socke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 scale=1 1 1
- link hexagon_socket_head_cap_screw_iso_4762___m2_x_10_steel_4_6_plain__11__1: geometry visual mesh filename=package://glove_non_diametric/meshes/hardware/Hexagon_Socke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 scale=1 1 1
- link hexagon_socket_head_cap_screw_iso_4762___m2_x_10_steel_4_6_plain__11__2: geometry visual mesh filename=package://glove_non_diametric/meshes/hardware/Hexagon_Socke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 scale=1 1 1
- link hexagon_socket_head_cap_screw_iso_4762___m2_x_10_steel_4_6_plain__11__3: geometry visual mesh filename=package://glove_non_diametric/meshes/hardware/Hexagon_Socke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 scale=1 1 1
- link hexagon_socket_head_cap_screw_iso_4762___m2_x_10_steel_4_6_plain__11__4: geometry visual mesh filename=package://glove_non_diametric/meshes/hardware/Hexagon_Socke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 scale=1 1 1
- link hexagon_socket_head_cap_screw_iso_4762___m2_x_10_steel_4_6_plain__12_: geometry visual mesh filename=package://glove_non_diametric/meshes/hardware/Hexagon_Socke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 scale=1 1 1
- link hexagon_socket_head_cap_screw_iso_4762___m2_x_10_steel_4_6_plain__13_: geometry visual mesh filename=package://glove_non_diametric/meshes/hardware/Hexagon_Socke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 scale=1 1 1
- link hexagon_socket_head_cap_screw_iso_4762___m2_x_10_steel_4_6_plain__14_: geometry visual mesh filename=package://glove_non_diametric/meshes/hardware/Hexagon_Socke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 scale=1 1 1
- link hexagon_socket_head_cap_screw_iso_4762___m2_x_10_steel_4_6_plain__15_: geometry visual mesh filename=package://glove_non_diametric/meshes/hardware/Hexagon_Socke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 scale=1 1 1
- link hexagon_socket_head_cap_screw_iso_4762___m2_x_10_steel_4_6_plain__16_: geometry visual mesh filename=package://glove_non_diametric/meshes/hardware/Hexagon_Socke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 scale=1 1 1
- link hexagon_socket_head_cap_screw_iso_4762___m2_x_10_steel_4_6_plain__17_: geometry visual mesh filename=package://glove_non_diametric/meshes/hardware/Hexagon_Socke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 scale=1 1 1
- link hexagon_socket_head_cap_screw_iso_4762___m2_x_10_steel_4_6_plain__18_: geometry visual mesh filename=package://glove_non_diametric/meshes/hardware/Hexagon_Socke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 scale=1 1 1
- link hexagon_socket_head_cap_screw_iso_4762___m2_x_10_steel_4_6_plain__19_: geometry visual mesh filename=package://glove_non_diametric/meshes/hardware/Hexagon_Socke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 scale=1 1 1
- link hexagon_socket_head_cap_screw_iso_4762___m2_x_10_steel_4_6_plain__1_: geometry visual mesh filename=package://glove_non_diametric/meshes/hardware/Hexagon_Socke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 scale=1 1 1
- link hexagon_socket_head_cap_screw_iso_4762___m2_x_10_steel_4_6_plain__2_: geometry visual mesh filename=package://glove_non_diametric/meshes/hardware/Hexagon_Socke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 scale=1 1 1
- link hexagon_socket_head_cap_screw_iso_4762___m2_x_10_steel_4_6_plain__3_: geometry visual mesh filename=package://glove_non_diametric/meshes/hardware/Hexagon_Socke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 scale=1 1 1
- link hexagon_socket_head_cap_screw_iso_4762___m2_x_10_steel_4_6_plain__4_: geometry visual mesh filename=package://glove_non_diametric/meshes/hardware/Hexagon_Socke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 scale=1 1 1
- link hexagon_socket_head_cap_screw_iso_4762___m2_x_10_steel_4_6_plain__5_: geometry visual mesh filename=package://glove_non_diametric/meshes/hardware/Hexagon_Socke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 scale=1 1 1
- link hexagon_socket_head_cap_screw_iso_4762___m2_x_10_steel_4_6_plain__6_: geometry visual mesh filename=package://glove_non_diametric/meshes/hardware/Hexagon_Socke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 scale=1 1 1
- link hexagon_socket_head_cap_screw_iso_4762___m2_x_10_steel_4_6_plain__7_: geometry visual mesh filename=package://glove_non_diametric/meshes/hardware/Hexagon_Socke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 scale=1 1 1
- link hexagon_socket_head_cap_screw_iso_4762___m2_x_10_steel_4_6_plain__8_: geometry visual mesh filename=package://glove_non_diametric/meshes/hardware/Hexagon_Socke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 scale=1 1 1
- link hexagon_socket_head_cap_screw_iso_4762___m2_x_10_steel_4_6_plain__9_: geometry visual mesh filename=package://glove_non_diametric/meshes/hardware/Hexagon_Socke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 scale=1 1 1
- link hexagon_socket_head_cap_screw_iso_4762___m2_x_12_steel_4_6_plain: geometry visual mesh filename=package://glove_non_diametric/meshes/hardware/Hexagon_Socke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 scale=1 1 1
- link hexagon_socket_head_cap_screw_iso_4762___m2_x_12_steel_4_6_plain__10_: geometry visual mesh filename=package://glove_non_diametric/meshes/hardware/Hexagon_Socke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 scale=1 1 1
- link hexagon_socket_head_cap_screw_iso_4762___m2_x_12_steel_4_6_plain__11_: geometry visual mesh filename=package://glove_non_diametric/meshes/hardware/Hexagon_Socke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 scale=1 1 1
- link hexagon_socket_head_cap_screw_iso_4762___m2_x_12_steel_4_6_plain__12_: geometry visual mesh filename=package://glove_non_diametric/meshes/hardware/Hexagon_Socke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 scale=1 1 1
- link hexagon_socket_head_cap_screw_iso_4762___m2_x_12_steel_4_6_plain__1_: geometry visual mesh filename=package://glove_non_diametric/meshes/hardware/Hexagon_Socke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 scale=1 1 1
- link hexagon_socket_head_cap_screw_iso_4762___m2_x_12_steel_4_6_plain__2_: geometry visual mesh filename=package://glove_non_diametric/meshes/hardware/Hexagon_Socke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 scale=1 1 1
- link hexagon_socket_head_cap_screw_iso_4762___m2_x_12_steel_4_6_plain__3_: geometry visual mesh filename=package://glove_non_diametric/meshes/hardware/Hexagon_Socke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 scale=1 1 1
- link hexagon_socket_head_cap_screw_iso_4762___m2_x_12_steel_4_6_plain__4_: geometry visual mesh filename=package://glove_non_diametric/meshes/hardware/Hexagon_Socke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 scale=1 1 1
- link hexagon_socket_head_cap_screw_iso_4762___m2_x_12_steel_4_6_plain__5_: geometry visual mesh filename=package://glove_non_diametric/meshes/hardware/Hexagon_Socke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 scale=1 1 1
- link hexagon_socket_head_cap_screw_iso_4762___m2_x_12_steel_4_6_plain__6_: geometry visual mesh filename=package://glove_non_diametric/meshes/hardware/Hexagon_Socke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 scale=1 1 1
- link hexagon_socket_head_cap_screw_iso_4762___m2_x_12_steel_4_6_plain__7_: geometry visual mesh filename=package://glove_non_diametric/meshes/hardware/Hexagon_Socke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 scale=1 1 1
- link hexagon_socket_head_cap_screw_iso_4762___m2_x_12_steel_4_6_plain__8_: geometry visual mesh filename=package://glove_non_diametric/meshes/hardware/Hexagon_Socke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 scale=1 1 1
- link hexagon_socket_head_cap_screw_iso_4762___m2_x_12_steel_4_6_plain__9_: geometry visual mesh filename=package://glove_non_diametric/meshes/hardware/Hexagon_Socke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 scale=1 1 1
- link hexagon_socket_head_cap_screw_iso_4762___m2_x_16_steel_4_6_plain: geometry visual mesh filename=package://glove_non_diametric/meshes/hardware/Hexagon_Socke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 scale=1 1 1
- link hexagon_socket_head_cap_screw_iso_4762___m2_x_16_steel_4_6_plain__1_: geometry visual mesh filename=package://glove_non_diametric/meshes/hardware/Hexagon_Socke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 scale=1 1 1
- link hexagon_socket_head_cap_screw_iso_4762___m2_x_16_steel_4_6_plain__2_: geometry visual mesh filename=package://glove_non_diametric/meshes/hardware/Hexagon_Socke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 scale=1 1 1
- link hexagon_socket_head_cap_screw_iso_4762___m2_x_16_steel_4_6_plain__3_: geometry visual mesh filename=package://glove_non_diametric/meshes/hardware/Hexagon_Socke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 scale=1 1 1
- link hexagon_socket_head_cap_screw_iso_4762___m2_x_6_steel_4_6_plain: geometry visual mesh filename=package://glove_non_diametric/meshes/hardware/Hexagon_Socke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 scale=1 1 1
- link hexagon_socket_head_cap_screw_iso_4762___m2_x_6_steel_4_6_plain__10_: geometry visual mesh filename=package://glove_non_diametric/meshes/hardware/Hexagon_Socke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 scale=1 1 1
- link hexagon_socket_head_cap_screw_iso_4762___m2_x_6_steel_4_6_plain__11_: geometry visual mesh filename=package://glove_non_diametric/meshes/hardware/Hexagon_Socke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 scale=1 1 1
- link hexagon_socket_head_cap_screw_iso_4762___m2_x_6_steel_4_6_plain__12_: geometry visual mesh filename=package://glove_non_diametric/meshes/hardware/Hexagon_Socke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 scale=1 1 1
- link hexagon_socket_head_cap_screw_iso_4762___m2_x_6_steel_4_6_plain__13_: geometry visual mesh filename=package://glove_non_diametric/meshes/hardware/Hexagon_Socke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 scale=1 1 1
- link hexagon_socket_head_cap_screw_iso_4762___m2_x_6_steel_4_6_plain__14_: geometry visual mesh filename=package://glove_non_diametric/meshes/hardware/Hexagon_Socke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 scale=1 1 1
- link hexagon_socket_head_cap_screw_iso_4762___m2_x_6_steel_4_6_plain__15_: geometry visual mesh filename=package://glove_non_diametric/meshes/hardware/Hexagon_Socke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 scale=1 1 1
- link hexagon_socket_head_cap_screw_iso_4762___m2_x_6_steel_4_6_plain__16_: geometry visual mesh filename=package://glove_non_diametric/meshes/hardware/Hexagon_Socke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 scale=1 1 1
- link hexagon_socket_head_cap_screw_iso_4762___m2_x_6_steel_4_6_plain__17_: geometry visual mesh filename=package://glove_non_diametric/meshes/hardware/Hexagon_Socke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 scale=1 1 1
- link hexagon_socket_head_cap_screw_iso_4762___m2_x_6_steel_4_6_plain__18_: geometry visual mesh filename=package://glove_non_diametric/meshes/hardware/Hexagon_Socke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 scale=1 1 1
- link hexagon_socket_head_cap_screw_iso_4762___m2_x_6_steel_4_6_plain__1_: geometry visual mesh filename=package://glove_non_diametric/meshes/hardware/Hexagon_Socke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 scale=1 1 1
- link hexagon_socket_head_cap_screw_iso_4762___m2_x_6_steel_4_6_plain__2_: geometry visual mesh filename=package://glove_non_diametric/meshes/hardware/Hexagon_Socke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 scale=1 1 1
- link hexagon_socket_head_cap_screw_iso_4762___m2_x_6_steel_4_6_plain__3_: geometry visual mesh filename=package://glove_non_diametric/meshes/hardware/Hexagon_Socke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 scale=1 1 1
- link hexagon_socket_head_cap_screw_iso_4762___m2_x_6_steel_4_6_plain__4_: geometry visual mesh filename=package://glove_non_diametric/meshes/hardware/Hexagon_Socke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 scale=1 1 1
- link hexagon_socket_head_cap_screw_iso_4762___m2_x_6_steel_4_6_plain__5_: geometry visual mesh filename=package://glove_non_diametric/meshes/hardware/Hexagon_Socke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 scale=1 1 1
- link hexagon_socket_head_cap_screw_iso_4762___m2_x_6_steel_4_6_plain__6_: geometry visual mesh filename=package://glove_non_diametric/meshes/hardware/Hexagon_Socke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 scale=1 1 1
- link hexagon_socket_head_cap_screw_iso_4762___m2_x_6_steel_4_6_plain__7_: geometry visual mesh filename=package://glove_non_diametric/meshes/hardware/Hexagon_Socke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 scale=1 1 1
- link hexagon_socket_head_cap_screw_iso_4762___m2_x_6_steel_4_6_plain__8_: geometry visual mesh filename=package://glove_non_diametric/meshes/hardware/Hexagon_Socke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 scale=1 1 1
- link hexagon_socket_head_cap_screw_iso_4762___m2_x_6_steel_4_6_plain__9_: geometry visual mesh filename=package://glove_non_diametric/meshes/hardware/Hexagon_Socke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 scale=1 1 1
- link hexagon_thin_nut_iso_4035___m2_steel_6_plain: geometry visual mesh filename=package://glove_non_diametric/meshes/hardware/Hexagon_Thin_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 scale=1 1 1
- link hexagon_thin_nut_iso_4035___m2_steel_6_plain__1_: geometry visual mesh filename=package://glove_non_diametric/meshes/hardware/Hexagon_Thin_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 scale=1 1 1
- link hexagon_thin_nut_iso_4035___m2_steel_6_plain__2_: geometry visual mesh filename=package://glove_non_diametric/meshes/hardware/Hexagon_Thin_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 scale=1 1 1
- link hexagon_thin_nut_iso_4035___m2_steel_6_plain__3_: geometry visual mesh filename=package://glove_non_diametric/meshes/hardware/Hexagon_Thin_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 scale=1 1 1
- link hexagon_thin_nut_iso_4035___m2_steel_6_plain__4_: geometry visual mesh filename=package://glove_non_diametric/meshes/hardware/Hexagon_Thin_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 scale=1 1 1
- link hexagon_thin_nut_iso_4035___m2_steel_6_plain__5_: geometry visual mesh filename=package://glove_non_diametric/meshes/hardware/Hexagon_Thin_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 scale=1 1 1
- link hexagon_thin_nut_iso_4035___m2_steel_6_plain__6_: geometry visual mesh filename=package://glove_non_diametric/meshes/hardware/Hexagon_Thin_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 scale=1 1 1
- link hexagon_thin_nut_iso_4035___m2_steel_6_plain__7_: geometry visual mesh filename=package://glove_non_diametric/meshes/hardware/Hexagon_Thin_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 scale=1 1 1
- link hexagon_thin_nut_iso_4036___m2_steel_6_plain: geometry visual mesh filename=package://glove_non_diametric/meshes/hardware/Hexagon_Thin_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 scale=1 1 1
- link hexagon_thin_nut_iso_4036___m2_steel_6_plain__1_: geometry visual mesh filename=package://glove_non_diametric/meshes/hardware/Hexagon_Thin_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 scale=1 1 1
- link index_dip_2: geometry visual mesh filename=package://glove_non_diametric/meshes/printed/DIP/index_dip_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 scale=1 1 1
- link index_dip_2_1: geometry visual mesh filename=package://glove_non_diametric/meshes/printed/DIP/index_dip_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 scale=1 1 1
- link index_dip_2_2: geometry visual mesh filename=package://glove_non_diametric/meshes/printed/DIP/index_dip_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 scale=1 1 1
- link index_pip_1: geometry visual mesh filename=package://glove_non_diametric/meshes/printed/PIP/index_pip_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 scale=1 1 1
- link index_pip_2: geometry visual mesh filename=package://glove_non_diametric/meshes/printed/PIP/index_pip_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 scale=1 1 1
- link mcp_1: geometry visual mesh filename=package://glove_non_diametric/meshes/printed/MCP/mcp_1.stl scale=1 1 1
- link mcp_1_1: geometry visual mesh filename=package://glove_non_diametric/meshes/printed/MCP/mcp_1.stl scale=1 1 1
- link mcp_1_2: geometry visual mesh filename=package://glove_non_diametric/meshes/printed/MCP/mcp_1.stl scale=1 1 1
- link mcp_1_3: geometry visual mesh filename=package://glove_non_diametric/meshes/printed/MCP/mcp_1.stl scale=1 1 1
- link mcp_1_4: geometry visual mesh filename=package://glove_non_diametric/meshes/printed/MCP/mcp_1.stl scale=1 1 1
- link mcp_2: geometry visual mesh filename=package://glove_non_diametric/meshes/printed/MCP/mcp_2.stl scale=1 1 1
- link mcp_2_1: geometry visual mesh filename=package://glove_non_diametric/meshes/printed/MCP/mcp_2.stl scale=1 1 1
- link mcp_2_2: geometry visual mesh filename=package://glove_non_diametric/meshes/printed/MCP/mcp_2.stl scale=1 1 1
- link mcp_2_3: geometry visual mesh filename=package://glove_non_diametric/meshes/printed/MCP/mcp_2.stl scale=1 1 1
- link mcp_2_4: geometry visual mesh filename=package://glove_non_diametric/meshes/printed/MCP/mcp_2.stl scale=1 1 1
- link mcp_3: geometry visual mesh filename=package://glove_non_diametric/meshes/printed/MCP/mcp_3.stl scale=1 1 1
- link mcp_3_1: geometry visual mesh filename=package://glove_non_diametric/meshes/printed/MCP/mcp_3_1.stl scale=1 1 1
- link mcp_3_2: geometry visual mesh filename=package://glove_non_diametric/meshes/printed/MCP/mcp_3.stl scale=1 1 1
- link mcp_3_3: geometry visual mesh filename=package://glove_non_diametric/meshes/printed/MCP/mcp_3_1.stl scale=1 1 1
- link mcp_3_4: geometry visual mesh filename=package://glove_non_diametric/meshes/printed/MCP/mcp_3_1.stl scale=1 1 1
- link mcp_3_5: geometry visual mesh filename=package://glove_non_diametric/meshes/printed/MCP/mcp_3.stl scale=1 1 1
- link mcp_3_6: geometry visual mesh filename=package://glove_non_diametric/meshes/printed/MCP/mcp_3_1.stl scale=1 1 1
- link mcp_3_7: geometry visual mesh filename=package://glove_non_diametric/meshes/printed/MCP/mcp_3.stl scale=1 1 1
- link mcp_3__1_: geometry visual mesh filename=package://glove_non_diametric/meshes/printed/MCP/mcp_3__1_.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 scale=1 1 1
- link mcp_3__1__1: geometry visual mesh filename=package://glove_non_diametric/meshes/printed/MCP/mcp_3__1__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 scale=1 1 1
- link middle_pip_1: geometry visual mesh filename=package://glove_non_diametric/meshes/printed/PIP/middle_pip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 scale=1 1 1
- link middle_pip_2: geometry visual mesh filename=package://glove_non_diametric/meshes/printed/PIP/middle_pip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 scale=1 1 1
- link pip_1: geometry visual mesh filename=package://glove_non_diametric/meshes/printed/PIP/pip_1.stl scale=1 1 1
- link pip_2: geometry visual mesh filename=package://glove_non_diametric/meshes/printed/PIP/pip_2.stl scale=1 1 1
- link ring_pip_1: geometry visual mesh filename=package://glove_non_diametric/meshes/printed/PIP/ring_pip_1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 scale=1 1 1
- link ring_pip_2: geometry visual mesh filename=package://glove_non_diametric/meshes/printed/PIP/ring_pip_2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 scale=1 1 1
- link root: geometry visual mesh filename=package://glove_non_diametric/meshes/electronics/C0402_L1_0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 scale=1 1 1; visual mesh filename=package://glove_non_diametric/meshes/electronics/C0402_L1_0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 scale=1 1 1
- link thumb_dip_1: geometry visual mesh filename=package://glove_non_diametric/meshes/printed/DIP/thumb_dip_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 scale=1 1 1
- link thumb_dip_2: geometry visual mesh filename=package://glove_non_diametric/meshes/printed/DIP/thumb_dip_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 scale=1 1 1
- link thumb_mount: geometry visual mesh filename=package://glove_non_diametric/meshes/printed/palm/thumb_mou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 scale=1 1 1
- link thumb_pip_1: geometry visual mesh filename=package://glove_non_diametric/meshes/printed/PIP/thumb_pip_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 scale=1 1 1
- link thumb_pip_2: geometry visual mesh filename=package://glove_non_diametric/meshes/printed/PIP/thumb_pip_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 scale=1 1 1
- link thumb_pip_4: geometry visual mesh filename=package://glove_non_diametric/meshes/printed/PIP/thumb_pip_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 scale=1 1 1
- link top_base: geometry visual mesh filename=package://glove_non_diametric/meshes/printed/palm/top_base.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 scale=1 1 1
